File: PCB/MerlynActionCam.kicad_pcb (KiCad board)
At the start: 2 copper layers, 16 parts, among them Q1 AO3401A, U1 TPS63802DLAR, U2 BQ25606RGER

Commit message: checkpoint
Parts:
- added C10: 10uF, Capacitor_SMD:C_0603_1608Metric, F.Cu at (124.6, 84.1)
- added C11: 10uF, Capacitor_SMD:C_0603_1608Metric, F.Cu at (124.6, 86.7)
- added C12: 22uF, Capacitor_SMD:C_0603_1608Metric, F.Cu at (128.6, 76.6)
- added C13: 10uF, Capacitor_SMD:C_0603_1608Metric, F.Cu at (128.6, 79.1)
- added C14: 10uF, Capacitor_SMD:C_0603_1608Metric, F.Cu at (128.6, 81.6)
- added C15: 22uF, Capacitor_SMD:C_0603_1608Metric, F.Cu at (128.6, 84.1)
- added C16: 10uF, Capacitor_SMD:C_0603_1608Metric, F.Cu at (128.6, 86.7)
- added C17: 0.1uF, Capacitor_SMD:C_0402_1005Metric, F.Cu at (129.0, 99.6)
- added C6: 10uF, Capacitor_SMD:C_0603_1608Metric, F.Cu at (124.6, 76.6)
- added C7: 1uF, Capacitor_SMD:C_0402_1005Metric, F.Cu at (129.0, 97.6)
- added C8: 10uF, Capacitor_SMD:C_0603_1608Metric, F.Cu at (124.6, 79.1)
- added C9: 22uF, Capacitor_SMD:C_0603_1608Metric, F.Cu at (124.6, 81.6)
- added CN1: OK-10F030-04, easyeda2kicad:CONN-SMD_30P-P0.40_OK-10F030-04-A, B.Cu at (116.1, 107.8)
- added FPC1: FPC-05F-22PH20, easyeda2kicad:FPC-SMD_22P-P0.50_FPC-05F-22PH20, B.Cu at (138.8, 101.6)
- added L2: 0.47uH, easyeda2kicad:L_Changjiang_FTC201610S, F.Cu at (143.3, 87.0)
- added L3: 1.5uH, easyeda2kicad:L_Changjiang_FTC201610S, F.Cu at (143.3, 90.3)
- added L4: 1.5uH, easyeda2kicad:L_Changjiang_FTC201610S, F.Cu at (143.3, 93.7)
- added LED1: YLED0602RSIDE, easyeda2kicad:LED-SMD_L1.6-W1.1-RD, F.Cu at (128.7, 91.6)
- added LED2: WHITE, easyeda2kicad:LED-SMD_L1.6-W1.1-R-RD_WHITE, F.Cu at (128.7, 89.3)
- added Q2: AO3401A, Package_TO_SOT_SMD:SOT-23, F.Cu at (144.7, 77.8)
- added Q3: AO3401A, Package_TO_SOT_SMD:SOT-23, F.Cu at (144.7, 82.4)
- added R10: 56k, Resistor_SMD:R_0402_1005Metric, F.Cu at (132.1, 84.3)
- added R11: 10k, Resistor_SMD:R_0402_1005Metric, F.Cu at (135.0, 76.3)
- added R12: 15k, Resistor_SMD:R_0402_1005Metric, F.Cu at (135.0, 78.3)
- added R13: 10k, Resistor_SMD:R_0402_1005Metric, F.Cu at (135.0, 80.3)
- added R14: 10k, Resistor_SMD:R_0402_1005Metric, F.Cu at (135.0, 82.3)
- added R15: 10k, Resistor_SMD:R_0402_1005Metric, F.Cu at (135.0, 84.3)
- added R16: 15k, Resistor_SMD:R_0402_1005Metric, F.Cu at (137.9, 76.3)
- added R17: 5.1k, Resistor_SMD:R_0402_1005Metric, F.Cu at (137.9, 78.3)
- added R18: 270R, Resistor_SMD:R_0402_1005Metric, F.Cu at (137.9, 80.3)
- added R19: 10k, Resistor_SMD:R_0402_1005Metric, F.Cu at (137.9, 82.3)
- added R20: 10k, Resistor_SMD:R_0402_1005Metric, F.Cu at (137.9, 84.3)
- added R21: 10k, Resistor_SMD:R_0402_1005Metric, F.Cu at (140.8, 76.3)
- added R22: 10k, Resistor_SMD:R_0402_1005Metric, F.Cu at (140.8, 78.3)
- added R23: 10k, Resistor_SMD:R_0402_1005Metric, F.Cu at (140.8, 80.3)
- added R24: 36k, Resistor_SMD:R_0402_1005Metric, F.Cu at (140.8, 82.3)
- added R25: 5.1k, Resistor_SMD:R_0402_1005Metric, F.Cu at (140.8, 84.3)
- added R6: 5.1k, Resistor_SMD:R_0402_1005Metric, F.Cu at (132.1, 76.3)
- added R7: 5.1k, Resistor_SMD:R_0402_1005Metric, F.Cu at (132.1, 78.3)
- added R8: 10k, Resistor_SMD:R_0402_1005Metric, F.Cu at (132.1, 80.3)
- added R9: 10k, Resistor_SMD:R_0402_1005Metric, F.Cu at (132.1, 82.3)
- added SW1: TS24CA, easyeda2kicad:SW-SMD_2P-TS24CA, F.Cu at (164.4, 95.3)
- added U3: RT8097CHGE, easyeda2kicad:SOT-23-6_L2.9-W1.6-P0.95-LS2.8-BL, F.Cu at (125.1, 90.1)
- added U4: RT8097CHGE, easyeda2kicad:SOT-23-6_L2.9-W1.6-P0.95-LS2.8-BL, F.Cu at (125.1, 94.5)
- added U5: CH32V003F4U6, easyeda2kicad:QFN-20_L3.0-W3.0-P0.40-TL-EP1.7, F.Cu at (125.2, 98.9)
- added USB1: TYPE-C 16PIN, easyeda2kicad:USB-C-SMD_TYPE-C-6PIN-2MD-073, F.Cu at (136.0, 88.7)
- moved 1 40.7 mm to (136.5, 109.8)
Connections:
- 1 pad 100: unconnected-(1-SR0_IO2-Pad100) -> MIPI_D0+
- 1 pad 101: unconnected-(1-SR0_IO3-Pad101) -> MIPI_D0-
- 1 pad 102: unconnected-(1-SR0_IO4-Pad102) -> MIPI_D1+
- 1 pad 103: unconnected-(1-SR0_IO5-Pad103) -> MIPI_D1-
- 1 pad 104: unconnected-(1-SR0_IO6-Pad104) -> MIPI_CLK+
- 1 pad 105: unconnected-(1-SR0_IO7-Pad105) -> MIPI_CLK-
- 1 pad 106: unconnected-(1-SR0_IO8-Pad106) -> MIPI_D2+
- 1 pad 107: unconnected-(1-SR0_IO9-Pad107) -> MIPI_D2-
- 1 pad 108: unconnected-(1-SR0_IO10-Pad108) -> MIPI_D3+
- 1 pad 109: unconnected-(1-SR0_IO11-Pad109) -> MIPI_D3-
- 1 pad 111: unconnected-(1-SR0_IO16-Pad111) -> MIPI_RST
- 1 pad 112: unconnected-(1-SR0_IO17-Pad112) -> MIPI_MCLK
- 1 pad 113: unconnected-(1-SR0_IO18-Pad113) -> SCL
- 1 pad 114: unconnected-(1-SR0_IO19-Pad114) -> SDA
- 1 pad 30: unconnected-(1-USB2_DM-Pad30) -> D-
- 1 pad 31: unconnected-(1-USB2_DP-Pad31) -> D+
- C3 pad 1: Net-(U2-VBUS) -> +5-14V
- C5 pad 1: unconnected-(C5-Pad1) -> Net-(U2-BTST)
- C5 pad 2: unconnected-(C5-Pad2) -> Net-(C5-Pad2)
- D1 pad 1: unconnected-(D1-K-Pad1) -> +5-14V
- D1 pad 2: unconnected-(D1-A-Pad2) -> Net-(D1-A)
- L1 pad 1: unconnected-(L1-Pad1) -> Net-(C5-Pad2)
- L1 pad 2: unconnected-(L1-Pad2) -> SYSTEM
- R1 pad 1: unconnected-(R1-Pad1) -> Net-(D1-A)
- R1 pad 2: unconnected-(R1-Pad2) -> GND
- U1 pad 1: unconnected-(U1-EN-Pad1) -> 1V5PG
- U1 pad 10: unconnected-(U1-VIN-Pad10) -> +BATT
- U1 pad 2: unconnected-(U1-MODE-Pad2) -> +BATT
- U1 pad 3: unconnected-(U1-AGND-Pad3) -> GND
- U1 pad 4: unconnected-(U1-FB-Pad4) -> Net-(U1-FB)
- U1 pad 6: unconnected-(U1-VOUT-Pad6) -> +3V3
- U1 pad 7: unconnected-(U1-L2-Pad7) -> Net-(U1-L2)
- U1 pad 8: unconnected-(U1-GND-Pad8) -> GND
- U1 pad 9: unconnected-(U1-L1-Pad9) -> Net-(U1-L1)
- U2 pad 15: Net-(U2-SYS-Pad15) -> SYSTEM
- U2 pad 16: Net-(U2-SYS-Pad15) -> SYSTEM
- U2 pad 17: unconnected-(U2-GND-Pad17) -> GND
- U2 pad 18: unconnected-(U2-GND-Pad18) -> GND
- U2 pad 19: unconnected-(U2-SW-Pad19) -> Net-(C5-Pad2)
- U2 pad 20: unconnected-(U2-SW-Pad20) -> Net-(C5-Pad2)
- U2 pad 21: BTST -> Net-(U2-BTST)
- U2 pad 24: Net-(U2-VBUS) -> +5-14V
- U2 pad 5: unconnected-(U2-STAT-Pad5) -> CHARGE
- U2 pad 7: unconnected-(U2-~{PG}-Pad7) -> PG
Routing:
- net MIPI_CLK-: track 0.00 -> 4.59 mm, vias 0 -> 1
- net MIPI_CLK+: track 0.00 -> 3.87 mm, vias 0 -> 1
Other:
- copper layers 2 -> 4

Commit message: checkpoint
Parts:
- CN1, FPC1: moved to F.Cu
- moved FPC1 50.5 mm to (90.3, 87.2)
- moved 1 20.0 mm to (120.1, 121.4)
- moved CN1 7.94 mm to (123.0, 111.7), turned to 180 degrees
Connections:
- 1 pad 100: MIPI_D0+ -> MIPI_D3+
- 1 pad 101: MIPI_D0- -> MIPI_D3-
- 1 pad 102: MIPI_D1+ -> MIPI_D2+
- 1 pad 103: MIPI_D1- -> MIPI_D2-
- 1 pad 106: MIPI_D2+ -> MIPI_D1+
- 1 pad 107: MIPI_D2- -> MIPI_D1-
- 1 pad 108: MIPI_D3+ -> MIPI_D0+
- 1 pad 109: MIPI_D3- -> MIPI_D0-

Commit message: checkpoint
Parts:
- removed FPC1: FPC-05F-22PH20, easyeda2kicad:FPC-SMD_22P-P0.50_FPC-05F-22PH20
- added BT1: BAT, easyeda2kicad:Battery, F.Cu at (117.5, 87.5)
- added C18: 22nF, Capacitor_SMD:C_0402_1005Metric, F.Cu at (109.3, 78.4)
- added C19: 1uF, Capacitor_SMD:C_0402_1005Metric, F.Cu at (109.3, 80.4)
- added C20: 1uF, Capacitor_SMD:C_0402_1005Metric, F.Cu at (109.3, 82.4)
- added C21: 0.1uF, Capacitor_SMD:C_0402_1005Metric, F.Cu at (109.3, 84.3)
- added C22: 0.1uF, Capacitor_SMD:C_0402_1005Metric, F.Cu at (109.3, 86.3)
- added C23: 0.1uF, Capacitor_SMD:C_0402_1005Metric, F.Cu at (109.3, 88.3)
- added C24: 0.1uF, Capacitor_SMD:C_0402_1005Metric, F.Cu at (112.2, 78.4)
- added C25: 8pF, Capacitor_SMD:C_0402_1005Metric, F.Cu at (112.2, 80.4)
- added C26: 0.1uF, Capacitor_SMD:C_0402_1005Metric, F.Cu at (112.2, 82.4)
- added C27: 8pF, Capacitor_SMD:C_0402_1005Metric, F.Cu at (112.2, 84.3)
- added C28: 0.1uF, Capacitor_SMD:C_0402_1005Metric, F.Cu at (112.2, 86.3)
- added C29: 10uF, Capacitor_SMD:C_0603_1608Metric, F.Cu at (209.5, 109.4)
- added C30: 0.1uF, Capacitor_SMD:C_0402_1005Metric, F.Cu at (112.2, 88.3)
- added C31: 10uF, Capacitor_SMD:C_0603_1608Metric, F.Cu at (118.5, 85.0)
- added C32: 0.1uF, Capacitor_SMD:C_0402_1005Metric, F.Cu at (115.0, 78.4)
- added C33: 0.1uF, Capacitor_SMD:C_0402_1005Metric, F.Cu at (115.0, 80.4)
- added C34: 0.1uF, Capacitor_SMD:C_0402_1005Metric, F.Cu at (115.0, 82.4)
- added C35: 0.1uF, Capacitor_SMD:C_0402_1005Metric, F.Cu at (115.0, 84.3)
- added C36: 0.1uF, Capacitor_SMD:C_0402_1005Metric, F.Cu at (115.0, 86.3)
- added C37: 0.1uF, Capacitor_SMD:C_0402_1005Metric, B.Cu at (210.8, 93.9)
- added C38: 0.1uF, Capacitor_SMD:C_0402_1005Metric, B.Cu at (213.3, 93.9)
- added C39: 0.1uF, Capacitor_SMD:C_0402_1005Metric, F.Cu at (232.2, 107.3)
- added C40: 0.1uF, Capacitor_SMD:C_0402_1005Metric, F.Cu at (232.2, 105.3)
- added C41: 0.1uF, Capacitor_SMD:C_0402_1005Metric, F.Cu at (232.2, 103.4)
- added C42: 0.1uF, Capacitor_SMD:C_0402_1005Metric, F.Cu at (232.2, 101.4)
- added C43: 0.1uF, Capacitor_SMD:C_0402_1005Metric, F.Cu at (232.2, 99.4)
- added C44: 10uF, Capacitor_SMD:C_0603_1608Metric, F.Cu at (197.2, 79.3)
- added C45: 10uF, Capacitor_SMD:C_0603_1608Metric, F.Cu at (235.6, 108.5)
- added C46: 0.1uF, Capacitor_SMD:C_0402_1005Metric, F.Cu at (229.3, 111.3)
- added C47: 0.1uF, Capacitor_SMD:C_0402_1005Metric, F.Cu at (229.3, 109.3)
- added C48: 0.1uF, Capacitor_SMD:C_0402_1005Metric, F.Cu at (229.3, 107.3)
- added C49: 0.1uF, Capacitor_SMD:C_0402_1005Metric, F.Cu at (229.3, 105.3)
- added C50: 10uF, Capacitor_SMD:C_0603_1608Metric, F.Cu at (235.6, 106.0)
- added C51: 0.1uF, Capacitor_SMD:C_0402_1005Metric, B.Cu at (214.6, 93.9)
- added C52: 0.1uF, Capacitor_SMD:C_0402_1005Metric, F.Cu at (229.3, 101.4)
- added C53: 0.1uF, Capacitor_SMD:C_0402_1005Metric, F.Cu at (229.3, 99.4)
- added C54: 0.1uF, Capacitor_SMD:C_0402_1005Metric, F.Cu at (226.4, 111.3)
- added C55: 0.1uF, Capacitor_SMD:C_0402_1005Metric, F.Cu at (226.4, 109.3)
- added C56: 0.1uF, Capacitor_SMD:C_0402_1005Metric, F.Cu at (226.4, 107.3)
- added C57: 0.1uF, Capacitor_SMD:C_0402_1005Metric, F.Cu at (226.4, 105.3)
- added C58: 10uF, Capacitor_SMD:C_0603_1608Metric, B.Cu at (212.1, 93.9)
- added C59: 10uF, Capacitor_SMD:C_0603_1608Metric, F.Cu at (235.6, 101.0)
- added C60: 10uF, Capacitor_SMD:C_0603_1608Metric, F.Cu at (235.6, 98.4)
- added C61: 10uF, Capacitor_SMD:C_0603_1608Metric, B.Cu at (215.8, 93.9)
- added H1: ~, easyeda2kicad:JST_SH_SM04B-SRSS-TB_1x04-1MP_P1.00mm_Horizontal, F.Cu at (179.2, 70.8)
- added JP1: ChargeEnable, easyeda2kicad:SolderJumper-2_P1.3mm_Open_TrianglePad1.0x1.5mm, F.Cu at (150.3, 97.2)
- added R26: 100k, Resistor_SMD:R_0402_1005Metric, F.Cu at (100.5, 95.4)
- added R27: 100k, Resistor_SMD:R_0402_1005Metric, F.Cu at (100.5, 97.4)
- added R28: 51k, Resistor_SMD:R_0402_1005Metric, F.Cu at (100.5, 99.3)
- added R29: 100k, Resistor_SMD:R_0402_1005Metric, F.Cu at (100.5, 101.3)
- added R30: 4.7k, Resistor_SMD:R_0402_1005Metric, F.Cu at (100.5, 103.3)
- added R31: 200k, Resistor_SMD:R_0402_1005Metric, F.Cu at (103.4, 95.4)
- added R32: 5.1k, Resistor_SMD:R_0402_1005Metric, F.Cu at (103.4, 97.4)
- added R33: 5.1k, Resistor_SMD:R_0402_1005Metric, F.Cu at (103.4, 99.3)
- added R34: 5.1k, Resistor_SMD:R_0402_1005Metric, F.Cu at (103.4, 101.3)
- added R35: 5.1k, Resistor_SMD:R_0402_1005Metric, F.Cu at (103.4, 103.3)
- added R36: 100R, Resistor_SMD:R_0402_1005Metric, F.Cu at (106.3, 95.4)
- added R37: 100R, Resistor_SMD:R_0402_1005Metric, F.Cu at (106.3, 97.4)
- added R38: 10k, Resistor_SMD:R_0402_1005Metric, F.Cu at (106.3, 99.3)
- added TP1: SWDIO, easyeda2kicad:TestPoint, F.Cu at (113.6, 100.3)
- added TP2: USART1_TX, easyeda2kicad:TestPoint, F.Cu at (113.6, 101.9)
- added TP3: UART_TX, easyeda2kicad:TestPoint, F.Cu at (113.6, 103.4)
- added TP4: UART_RX, easyeda2kicad:TestPoint, F.Cu at (113.6, 104.9)
- added U10: W25Q128JVSIQTR, easyeda2kicad:SOIC-8_L5.3-W5.3-P1.27-LS8.0-BL, F.Cu at (199.3, 83.6)
- added U11: TF-115-BCP9, easyeda2kicad:TF-SMD_TF-115-BCP9, F.Cu at (193.3, 99.6)
- added U6: RT9193-18GB, easyeda2kicad:SOT-23-5_L3.0-W1.7-P0.95-LS2.8-BR, F.Cu at (116.9, 95.9)
- added U7: ICS43434, easyeda2kicad:MIC-SMD_6P-L3.5-W2.7-P0.90-BL, F.Cu at (204.7, 102.0)
- added U8: BMI270, easyeda2kicad:LGA-14_L3.0-W2.5-P0.50-BR, F.Cu at (116.7, 99.9)
- added U9: INMP441, easyeda2kicad:MIC-SMD_INMP441, F.Cu at (200.9, 104.2)
- added X1: 24MHz, easyeda2kicad:CRYSTAL-SMD_4P-L2.0-W1.6-BL, F.Cu at (118.7, 79.2)
- USB1: moved to B.Cu
- moved C9 107.6 mm to (232.2, 79.7)
- moved C8 107.0 mm to (231.4, 85.4)
- moved C10 104.6 mm to (229.2, 80.7), turned to 180 degrees
- moved R10 99.7 mm to (231.7, 81.0), turned to 180 degrees
- moved R11 98.3 mm to (233.1, 82.5), turned to 90 degrees
- moved U4 97.8 mm to (222.3, 83.3), turned to -90 degrees
- moved CN1 97.6 mm to (218.5, 91.4)
- moved U12 97.3 mm to (215.2, 100.5)
- moved C14 96.2 mm to (224.8, 83.3), turned to 90 degrees
- moved C15 96.0 mm to (224.6, 85.7)
- moved C16 91.2 mm to (219.7, 82.6), turned to -90 degrees
- moved C11 91.1 mm to (215.7, 82.7), turned to 90 degrees
- moved R14 91.1 mm to (226.0, 83.9), turned to -90 degrees
- moved R15 89.3 mm to (224.3, 81.3), turned to 180 degrees
- moved U3 88.4 mm to (213.2, 82.8), turned to -90 degrees
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- renumbered 1 to U12
Connections:
- CN1 pad 31: unconnected-(CN1-Pad31) -> GND
- CN1 pad 32: unconnected-(CN1-Pad32) -> GND
- CN1 pad 33: unconnected-(CN1-Pad33) -> GND
- CN1 pad 34: unconnected-(CN1-Pad34) -> GND
- CN1 pad 9: unconnected-(CN1-Pad9) -> Net-(CN1-Pad9)
- LED1 pad 1: unconnected-(LED1-K-Pad1) -> Net-(LED1-K)
- Q2 pad 3: Net-(BT2-+) -> +5-14VRP
- R25 pad 2: unconnected-(R25-Pad2) -> +3V3
- U12 pad 1: unconnected-(1-SPI_CK-Pad1) -> SPI_SCK
- U12 pad 10: unconnected-(1-SD0_CLK-Pad10) -> SD_CLK
- U12 pad 11: unconnected-(1-SD0_CMD-Pad11) -> SD_CMD
- U12 pad 115: unconnected-(1-VDD-Pad115) -> +1V0
- U12 pad 116: unconnected-(1-AVDD_XTAL-Pad116) -> +3V3
- U12 pad 117: unconnected-(1-XTAL_IN-Pad117) -> Net-(U12-XTAL_IN)
- U12 pad 118: unconnected-(1-XTAL_OUT-Pad118) -> Net-(U12-XTAL_OUT)
- U12 pad 12: unconnected-(1-SD0_D3-Pad12) -> SD_DATA3
- U12 pad 120: unconnected-(1-VDD-Pad120) -> +1V0
- U12 pad 127: unconnected-(1-VDDP_0-Pad127) -> +3V3
- U12 pad 128: unconnected-(1-SPI_CZ-Pad128) -> SPI_CZ
- U12 pad 129: unconnected-(1-EP-Pad129) -> GND
- U12 pad 13: unconnected-(1-SD0_D2-Pad13) -> SD_DATA2
- U12 pad 15: unconnected-(1-I2S0_BCK-Pad15) -> I2S0_BCK
- U12 pad 16: unconnected-(1-I2S0_WCK-Pad16) -> I2S0_WCK
- U12 pad 17: unconnected-(1-I2S0_DI-Pad17) -> I2S0_DI
- U12 pad 2: unconnected-(1-SPI_DI-Pad2) -> SPI_SDI
- U12 pad 23: unconnected-(1-VDD-Pad23) -> +1V0
- U12 pad 24: unconnected-(1-VDD_ETH-Pad24) -> +3V3
- U12 pad 29: unconnected-(1-AVDD3P3_USB-Pad29) -> +3V3
- U12 pad 3: unconnected-(1-SPI_DO-Pad3) -> SPI_SDO
- U12 pad 32: unconnected-(1-AVDD_AUD-Pad32) -> +3V3
- U12 pad 33: unconnected-(1-AUD_AVG-Pad33) -> Net-(U12-AUD_AVG)
- U12 pad 34: unconnected-(1-AUD_VRM_ADC-Pad34) -> GND
- U12 pad 4: unconnected-(1-SPI_WPZ-Pad4) -> SPI_WPZ
- U12 pad 40: unconnected-(1-AVDDIO_DRAM-Pad40) -> +1V5
- U12 pad 41: unconnected-(1-AVDDIO_DATA-Pad41) -> +1V5
- U12 pad 42: unconnected-(1-AVDD_PLL-Pad42) -> +3V3
- U12 pad 43: unconnected-(1-DVDD_DDR_RX-Pad43) -> Net-(U12-DVDD_DDR_RX)
- U12 pad 44: unconnected-(1-DVDD_DDR-Pad44) -> +1V0
- U12 pad 45: unconnected-(1-VDD-Pad45) -> +1V0
- U12 pad 46: unconnected-(1-VDDIO_DATA-Pad46) -> +1V5
- U12 pad 47: unconnected-(1-VDD-Pad47) -> +1V0
- U12 pad 48: unconnected-(1-VDDIO_MCLK-Pad48) -> +1V5
- U12 pad 49: unconnected-(1-VDDIO_DRAM-Pad49) -> +1V5
- U12 pad 5: unconnected-(1-SPI_HLD-Pad5) -> SPI_HLD
- U12 pad 50: unconnected-(1-PM_UART_RX-Pad50) -> Net-(U12-PM_UART_RX)
- U12 pad 51: unconnected-(1-PM_UART_TX-Pad51) -> Net-(U12-PM_UART_TX)
- U12 pad 54: unconnected-(1-PM_I2CM_SCL-Pad54) -> PM_I2CM_SCL
- U12 pad 55: unconnected-(1-PM_I2CM_SDA-Pad55) -> PM_I2CM_SDA
- U12 pad 56: unconnected-(1-PM_GPIO0-Pad56) -> Net-(LED1-K)
- U12 pad 57: unconnected-(1-PM_GPIO1-Pad57) -> REC_SIGNAL
- U12 pad 62: unconnected-(1-PM_GPIO6-Pad62) -> Net-(U12-PM_GPIO6)
- U12 pad 64: unconnected-(1-PM_GPIO8-Pad64) -> Net-(U12-PM_GPIO8)
- U12 pad 65: unconnected-(1-AVDD_NODIE-Pad65) -> +3V3
- U12 pad 67: unconnected-(1-PM_SPI_CK-Pad67) -> Net-(U12-PM_SPI_CK)
- U12 pad 7: unconnected-(1-SD0_CDZ-Pad7) -> SD_CDZ
- U12 pad 70: unconnected-(1-PM_SPI_WPZ-Pad70) -> Net-(U12-PM_SPI_WPZ)
- U12 pad 72: unconnected-(1-AVDD_PM_SPI-Pad72) -> +3V3
- U12 pad 73: unconnected-(1-DVDD_NODIE-Pad73) -> Net-(U12-DVDD_NODIE)
- U12 pad 8: unconnected-(1-SD0_D1-Pad8) -> SD_DATA1
- U12 pad 83: unconnected-(1-RESET-Pad83) -> Net-(U12-RESET)
- U12 pad 84: unconnected-(1-AVDD_RTC-Pad84) -> +3V3
- U12 pad 85: unconnected-(1-XTAL_IN_32K-Pad85) -> Net-(U12-XTAL_IN_32K)
- U12 pad 86: unconnected-(1-XTAL_OUT_32K-Pad86) -> Net-(U12-XTAL_OUT_32K)
- U12 pad 87: unconnected-(1-VDD-Pad87) -> +1V0
- U12 pad 88: unconnected-(1-VDD-Pad88) -> +1V0
- U12 pad 89: unconnected-(1-VDDP_1-Pad89) -> +3V3
- U12 pad 9: unconnected-(1-SD0_D0-Pad9) -> SD_DATA0
- U12 pad 90: unconnected-(1-FUART_RX-Pad90) -> Net-(H1-RX)
- U12 pad 91: unconnected-(1-FUART_TX-Pad91) -> Net-(H1-TX)
- U12 pad 96: unconnected-(1-VDD-Pad96) -> +1V0
- U12 pad 97: unconnected-(1-VDDP_2A-Pad97) -> +1V8
Routing:
- net +3V3: track 0.00 -> 17.0 mm, vias 0 -> 2
- net SD_CDZ: track 0.00 -> 12.3 mm
- net +1V0: track 0.00 -> 12.1 mm, vias 0 -> 1
- net SD_DATA1: track 0.00 -> 12.0 mm
- net SD_DATA0: track 0.00 -> 11.7 mm
- net SD_DATA2: track 0.00 -> 11.7 mm
- net SD_DATA3: track 0.00 -> 11.4 mm
- net SD_CMD: track 0.00 -> 11.1 mm
- net SD_CLK: track 0.00 -> 10.9 mm
- net +1V5: track 0.00 -> 8.92 mm
- net +BATT: track 0.00 -> 6.44 mm
- net GND: track 0.00 -> 2.86 mm
- net Net-(U1-FB): track 0.00 -> 2.72 mm
- net MIPI_D3+: track 0.00 -> 2.66 mm
- net MIPI_D3-: track 0.00 -> 2.64 mm
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- added copper zone on B.Cu, net GND
- added copper zone on F.Cu, net GND
- added copper zone on In1.Cu, net GND
Other:
- board outline added: 55.5 x 38 mm
