File: PCB/MerlynActionCam.kicad_pcb (KiCad board)
At the start: 4 copper layers, 55.5 x 38 mm, 130 parts, among them CN1 OK-10F030-04, Q1 AO3401A, Q2 AO3401A, Q3 AO3401A, SW1 TS24CA, U1 TPS63802DLAR, U10 W25Q128JVSIQTR, U11 TF-115-BCP9, U2 BQ25606RGER, U3 RT8097CHGE, U4 RT8097CHGE, U5 CH32V003F4U6, U6 RT9193-18GB, U7 ICS43434, U8 BMI270, U9 INMP441, X1 24MHz

Commit message: checkpoint
Parts:
- added REF**: MountingHole, easyeda2kicad:MountingHole, F.Cu at (186.5, 80.0)
- added REF**: MountingHole, easyeda2kicad:MountingHole, F.Cu at (186.5, 112.0)
- H1, TP3, TP4: moved to B.Cu
- moved C54 68.8 mm to (223.7, 94.7), turned to 0 degrees
- moved C53 64.3 mm to (223.7, 96.7), turned to 0 degrees
- moved C41 61.8 mm to (223.7, 95.7), turned to 0 degrees
- moved C40 61.5 mm to (223.7, 105.5), turned to 0 degrees
- moved R33 60.4 mm to (219.0, 88.7), turned to 180 degrees
- moved R32 59.6 mm to (220.9, 88.7)
- moved L1 59.1 mm to (190.4, 83.2), turned to 90 degrees
- moved R38 58.5 mm to (217.0, 88.7), turned to 180 degrees
- moved C6 58.3 mm to (193.0, 81.9), turned to 90 degrees
- moved C5 57.1 mm to (190.1, 85.3), turned to 180 degrees
- moved C1 57.0 mm to (194.6, 81.9), turned to 90 degrees
- moved BT1 56.3 mm to (196.5, 81.3), turned to 180 degrees
- moved Q2 56.2 mm to (188.5, 87.6), turned to 180 degrees
- moved R29 56.0 mm to (223.7, 100.6)
- moved R1 55.1 mm to (188.7, 88.5), turned to 90 degrees
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Routing:
- net +BATT: track 6.44 -> 54.8 mm, vias 0 -> 11
- net +3V3: track 26.6 -> 63.6 mm, vias 5 -> 10
- net Net-(H1-RX): track 0.00 -> 27.8 mm, vias 0 -> 2
- net Net-(H1-TX): track 0.00 -> 27.2 mm, vias 0 -> 2
- net SYSTEM: track 4.89 -> 26.3 mm, vias 0 -> 4
- net GND: track 33.7 -> 52.9 mm, vias 6 -> 64
- net SDA: track 0.00 -> 13.1 mm
- net SCL: track 0.00 -> 11.6 mm
- net Net-(Q1-S): track 0.00 -> 9.42 mm
- net MIPI_RST: track 0.00 -> 8.97 mm, vias 0 -> 2
- net MIPI_MCLK: track 0.00 -> 8.71 mm, vias 0 -> 2
- net Net-(LED1-K): track 0.00 -> 8.48 mm, vias 0 -> 2
- net REC_SIGNAL: track 0.00 -> 5.03 mm
- net +1V0: track 19.9 -> 24.8 mm
- net Net-(BT1-+): track 0.00 -> 4.27 mm, vias 0 -> 3
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
Commit message: checkpoint
Parts:
- removed C59: 10uF, Capacitor_SMD:C_0603_1608Metric
- added C22: 10uF, Capacitor_SMD:C_0603_1608Metric, B.Cu at (208.3, 105.3)
- added R27: 100R, Resistor_SMD:R_0402_1005Metric, B.Cu at (209.3, 107.5)
- added REF**: MountingHole, easyeda2kicad:MountingHole, F.Cu at (225.5, 112.0)
- added REF**: MountingHole, easyeda2kicad:MountingHole, F.Cu at (225.5, 80.0)
- C43, C50, C55: moved to B.Cu
- moved C48 58.1 mm to (214.0, 86.1), turned to 0 degrees
- moved C49 56.3 mm to (210.3, 79.7)
- moved C42 54.1 mm to (215.1, 88.7)
- moved C55 52.6 mm to (208.9, 103.1)
- moved C56 52.5 mm to (202.1, 79.8)
- moved C57 50.6 mm to (204.2, 86.9), turned to 0 degrees
- moved C43 47.1 mm to (208.9, 104.1)
- moved C3 45.4 mm to (194.5, 109.9)
- moved C28 43.1 mm to (206.1, 87.2), turned to 45 degrees
- moved C50 42.7 mm to (208.3, 101.9)
- moved C17 39.1 mm to (202.1, 107.7), turned to 90 degrees
- moved R19 31.9 mm to (201.1, 107.7), turned to 90 degrees
- moved C31 22.7 mm to (205.6, 106.1), turned to 180 degrees
- moved C44 18.1 mm to (214.6, 87.4)
- moved C32 16.2 mm to (207.6, 106.3), turned to -90 degrees
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Connections:
- C29 pad 2: GND -> Net-(U12-AUD_VRM_ADC)
- U12 pad 34: GND -> Net-(U12-AUD_VRM_ADC)
Routing:
- net +3V3: track 63.6 -> 174.9 mm, vias 10 -> 19
- net +1V0: track 24.8 -> 78.2 mm, vias 1 -> 7
- net +1V5: track 16.1 -> 65.5 mm, vias 0 -> 5
- net SYSTEM: track 26.3 -> 69.7 mm, vias 4 -> 6
- net +1V8: track 4.02 -> 42.9 mm, vias 3 -> 4
- net Net-(Q3-G): track 0.00 -> 38.0 mm, vias 0 -> 2
- net GND: track 52.9 -> 81.3 mm, vias 64 -> 115
- net CHARGE: track 1.67 -> 28.6 mm, vias 1 -> 2
- net PG: track 2.55 -> 28.5 mm, vias 1 -> 2
- net +5-14V: track 13.2 -> 37.4 mm, vias 1 -> 5
- net +5-14VRP: track 0.00 -> 18.6 mm, vias 0 -> 2
- net REC_SIGNAL: track 5.03 -> 22.3 mm
- net Net-(U12-AUD_VRM_ADC): track 0.00 -> 4.24 mm, vias 0 -> 2
- net SDA: track 13.1 -> 11.8 mm, vias 0 -> 2
- net Net-(U5-PC1): track 0.00 -> 1.00 mm
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- added copper zone on In2.Cu, net GND
Other:
- board size 55.5 x 38 mm -> 45 x 38 mm
