File: PCB/_autosave-MerlynActionCam.kicad_pcb (KiCad board)
At the start: 4 copper layers, 55.5 x 38 mm, 130 parts, among them CN1 OK-10F030-04, Q1 AO3401A, Q2 AO3401A, Q3 AO3401A, SW1 TS24CA, U1 TPS63802DLAR, U10 W25Q128JVSIQTR, U11 TF-115-BCP9, U2 BQ25606RGER, U3 RT8097CHGE, U4 RT8097CHGE, U5 CH32V003F4U6, U6 RT9193-18GB, U7 ICS43434, U8 BMI270, U9 INMP441, X1 24MHz

Commit message: checkpoint
Parts:
- moved C54 68.8 mm to (223.7, 94.7), turned to 0 degrees
- moved C53 64.3 mm to (223.7, 96.7), turned to 0 degrees
- moved C41 61.8 mm to (223.7, 95.7), turned to 0 degrees
- moved C40 61.5 mm to (223.7, 105.5), turned to 0 degrees
- moved R29 56.0 mm to (223.7, 100.6)
- moved R35 52.7 mm to (223.7, 104.5), turned to 180 degrees
- moved R30 52.2 mm to (223.7, 107.5)
- moved R34 51.9 mm to (223.7, 103.5), turned to 180 degrees
- moved R37 51.0 mm to (223.7, 98.6)
- moved R36 50.1 mm to (223.7, 97.7)
- moved R31 45.1 mm to (223.7, 106.5)
- moved C30 37.7 mm to (223.7, 101.6), turned to 180 degrees
- moved C35 34.5 mm to (223.7, 99.6), turned to 180 degrees
- moved C36 33.7 mm to (223.7, 102.6)
Routing:
- net Net-(LED1-K): track 0.00 -> 8.48 mm, vias 0 -> 2
- net +3V3: track 26.6 -> 34.2 mm
- net REC_SIGNAL: track 0.00 -> 5.03 mm
- net +1V0: track 19.9 -> 24.8 mm
- net Net-(U12-PM_GPIO6): track 0.00 -> 3.89 mm
- net Net-(U12-RESET): track 0.00 -> 3.46 mm
- net Net-(U12-DVDD_NODIE): track 0.00 -> 2.72 mm
- net Net-(U12-PM_GPIO8): track 0.00 -> 2.61 mm
- net Net-(U12-XTAL_OUT_32K): track 0.00 -> 2.45 mm
- net Net-(U12-PM_SPI_CK): track 0.00 -> 2.36 mm
- net Net-(U12-PM_SPI_WPZ): track 0.00 -> 2.33 mm
- net Net-(U12-XTAL_IN_32K): track 0.00 -> 2.19 mm
