File: PCB/MerlynActionCam.kicad_sch (KiCad schematic)
At the start: 35 parts, among them Q1 AO3401A, Q2 AO3401A, SW1 Switch, U1 TPS63802DLAR, U2 BQ25606RGER, U3 RT8097CHGE

Commit message: checkpoint
Parts:
- removed SW1: Switch, symbol Switch:SW_Push
- added C11, C13, C14, C16: 10uF, Capacitor_SMD:C_0603_1608Metric, symbol Device:C_Small
- added C12, C15: 22uF, Capacitor_SMD:C_0603_1608Metric, symbol Device:C_Small
- added C17: 0.1uF, Capacitor_SMD:C_0402_1005Metric, symbol Device:C_Small
- added L3, L4: 1.5uH, easyeda2kicad:L_Changjiang_FTC201610S, symbol Device:L_Small
- added LED1: YLED0602RSIDE, easyeda2kicad:LED-SMD_L1.6-W1.1-RD, symbol MerlynActionCam:YLED0602RSIDE
- added LED2: WHITE, easyeda2kicad:LED-SMD_L1.6-W1.1-R-RD_WHITE, symbol MerlynActionCam:YLED0602WSIDE
- added Q3: AO3401A, Package_TO_SOT_SMD:SOT-23, symbol Transistor_FET:AO3401A
- added R12, R16: 15k, Resistor_SMD:R_0402_1005Metric, symbol Device:R_Small
- added R13, R14, R15, R19, R20, R21, R22, R23: 10k, Resistor_SMD:R_0402_1005Metric, symbol Device:R_Small
- added R17, R25: 5.1k, Resistor_SMD:R_0402_1005Metric, symbol Device:R_Small
- added R18: 270R, Resistor_SMD:R_0402_1005Metric, symbol Device:R_Small
- added R24: 36k, Resistor_SMD:R_0402_1005Metric, symbol Device:R_Small
- added SW1: TS24CA, easyeda2kicad:SW-SMD_2P-TS24CA, symbol MerlynActionCam:TS24CA
- added TP1: SWDIO, symbol Connector:TestPoint
- added TP2: USART1_TX, symbol Connector:TestPoint
- added U4: RT8097CHGE, easyeda2kicad:SOT-23-6_L2.9-W1.6-P0.95-LS2.8-BL, symbol MerlynActionCam:RT8097CHGE
- added U5: CH32V003F4U6, easyeda2kicad:QFN-20_L3.0-W3.0-P0.40-TL-EP1.7, symbol MerlynActionCam:CH32V003F4U6
- USB1: value TYPE-C 16PIN 2MD(073) -> TYPE-C 16PIN
Connections:
- net GND: now also U3.2 (GND), C11.2, C12.2, C13.2, C14.2, C15.2, C16.2, C17.2, R12.1, R15.1, R20.2, R24.1, SW1.2, SW1.3, SW1.4, U4.2 (GND), U5.21 (VSS), U5.4 (VSS)
- net SYSTEM: now also C6.1, L1.2, U2.15 (SYS), U2.16 (SYS), C17.1, Q3.2 (S), R17.1, R19.2, R21.2, R22.2, U5.6 (VDD); no longer C8.1, R9.2, U1.10 (VIN), U1.2 (MODE)
- net CHARGE: now reaches U2.5 (STAT)
- net CHARGE: now also R21.1, U5.10 (PC3)
- net PG: now reaches U2.7 (~{PG})
- net PG: now also R22.1, U5.9 (PC2)
- net +BATT: now reaches U3.1 (EN)
- net +BATT: now also C8.1, R9.2, U1.10 (VIN), U1.2 (MODE), U3.4 (VIN), C11.1, C14.1, Q3.3 (D), R14.2, U4.4 (VIN)
- net at U3.3 (LX): now also L3.1
- net at U3.6 (FB): now also R12.2, R13.1
- net 1VPGOOD renamed 1V0PG
- net 1V0PG: now also U4.1 (EN); no longer U1.1 (EN)
- net 3V3FB: no longer names the net of R10.1, R11.2, U1.4 (FB)
- new net: R23.2, U5.12 (PC5)
- new net: R18.1, U5.8 (PC1)
- new net: Q3.1 (G), R18.2, R19.1
- new net: SW1.1, U5.11 (PC4)
- new net: LED1.2 (A), R25.1
- new net: LED2.1 (A), R17.2
- new net: LED2.2 (C), U5.18 (PD4)
- new net: R15.2, R16.1, U4.6 (FB)
- new net: R20.1, TP1.1, U5.15 (PD1)
- new net: L4.1, U4.3 (LX)
- new net: TP2.1, U5.19 (PD5)
- new net +1V0: C12.1, C13.1, L3.2, R13.2
- new net +1V5: C15.1, C16.1, L4.2, R16.2
- new net 1V5PG: R14.1, U1.1 (EN), U4.5 (PG)
- new net REC_SIGNAL: R23.1, R24.2
- no-connect marks 9 -> 17
Other:
- note added: "1.0V Regulator"
- note added: "1.5V Regulator"
- note added: "3.3V Regulator"
- note added: "Input Power & Battery Management"
- note added: "Power Switch, Button Handling, Battery Monitor"
- note added: "USB-C Port"
- note removed: "1.0V"
- note removed: "3.3V"
- note removed: "Battery"
- moved on the sheet: BT1, BT2, C1, C10, C2, C3, C4, C5, C6, C7, C8, C9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

Commit message: checkpoint
Parts:
- added CN1: OK-10F030-04, easyeda2kicad:CONN-SMD_30P-P0.40_OK-10F030-04-A, symbol MerlynActionCam:OK-10F030-04
- added FPC1: FPC-05F-22PH20, easyeda2kicad:FPC-SMD_22P-P0.50_FPC-05F-22PH20, symbol MerlynActionCam:FPC-05F-22PH20
Connections:
- net +3V3: now also CN1.13, CN1.14, FPC1.22
- net GND: now also CN1.1, CN1.10, CN1.12, CN1.15, CN1.18, CN1.21, CN1.24, CN1.27, CN1.3, CN1.30, FPC1.1, FPC1.10, FPC1.13, FPC1.16, FPC1.19, FPC1.4, FPC1.7
- net MIPI_D0+: now reaches 1.100 (SR0_IO2)
- net MIPI_D0+: now also CN1.17, FPC1.3
- net MIPI_D0-: now reaches 1.101 (SR0_IO3)
- net MIPI_D0-: now also CN1.16, FPC1.2
- net MIPI_D1+: now reaches 1.102 (SR0_IO4)
- net MIPI_D1+: now also CN1.20, FPC1.6
- net MIPI_D1-: now reaches 1.103 (SR0_IO5)
- net MIPI_D1-: now also CN1.19, FPC1.5
- net MIPI_CLK+: now reaches 1.104 (SR0_IO6)
- net MIPI_CLK+: now also CN1.23, FPC1.9
- net MIPI_CLK-: now reaches 1.105 (SR0_IO7)
- net MIPI_CLK-: now also CN1.22, FPC1.8
- net MIPI_D2+: now reaches 1.106 (SR0_IO8)
- net MIPI_D2+: now also CN1.26, FPC1.12
- net MIPI_D2-: now reaches 1.107 (SR0_IO9)
- net MIPI_D2-: now also CN1.25, FPC1.11
- net MIPI_D3+: now reaches 1.108 (SR0_IO10)
- net MIPI_D3+: now also CN1.29, FPC1.15
- net MIPI_D3-: now reaches 1.109 (SR0_IO11)
- net MIPI_D3-: now also CN1.28, FPC1.14
- net MIPI_RST: now reaches 1.111 (SR0_IO16)
- net MIPI_RST: now also CN1.8, FPC1.17
- net MIPI_MCLK: now reaches 1.112 (SR0_IO17)
- net MIPI_MCLK: now also CN1.11, FPC1.18
- net SCL: now reaches 1.113 (SR0_IO18)
- net SCL: now also CN1.4, FPC1.20
- net SDA: now reaches 1.114 (SR0_IO19)
- net SDA: now also CN1.5, FPC1.21
- no-connect marks 17 -> 21

Commit message: checkpoint
Parts:
- removed FPC1: FPC-05F-22PH20, easyeda2kicad:FPC-SMD_22P-P0.50_FPC-05F-22PH20, symbol MerlynActionCam:FPC-05F-22PH20
- added C18: 22nF, Capacitor_SMD:C_0402_1005Metric, symbol Device:C_Small
- added C19, C20: 1uF, Capacitor_SMD:C_0402_1005Metric, symbol Device:C_Small
- added C21, C22, C23, C24, C26, C28, C30, C32, C33, C34, C35, C36: 0.1uF, Capacitor_SMD:C_0402_1005Metric, symbol Device:C_Small
- added C25, C27: 8pF, Capacitor_SMD:C_0402_1005Metric, symbol Device:C_Small
- added C29, C31: 10uF, Capacitor_SMD:C_0603_1608Metric, symbol Device:C_Small
- added H1: ~, easyeda2kicad:JST_SH_SM04B-SRSS-TB_1x04-1MP_P1.00mm_Horizontal, symbol MerlynActionCam:MAVLINK
- added R26, R27, R29: 100k, Resistor_SMD:R_0402_1005Metric, symbol Device:R_Small
- added R28: 51k, Resistor_SMD:R_0402_1005Metric, symbol Device:R_Small
- added R30: 4.7k, Resistor_SMD:R_0402_1005Metric, symbol Device:R_Small
- added R31: 200k, Resistor_SMD:R_0402_1005Metric, symbol Device:R_Small
- added R32, R33, R34, R35: 5.1k, Resistor_SMD:R_0402_1005Metric, symbol Device:R_Small
- added R36, R37: 100R, Resistor_SMD:R_0402_1005Metric, symbol Device:R_Small
- added R38: 10k, Resistor_SMD:R_0402_1005Metric, symbol Device:R_Small
- added TP3: UART_TX, easyeda2kicad:TestPoint, symbol Connector:TestPoint
- added TP4: UART_RX, easyeda2kicad:TestPoint, symbol Connector:TestPoint
- added U10: W25Q128JVSIQTR, easyeda2kicad:SOIC-8_L5.3-W5.3-P1.27-LS8.0-BL, symbol MerlynActionCam:W25Q128JVSIQTR
- added U11: TF-115-BCP9, easyeda2kicad:TF-SMD_TF-115-BCP9, symbol MerlynActionCam:TF-115-BCP9
- added U6: RT9193-18GB, easyeda2kicad:SOT-23-5_L3.0-W1.7-P0.95-LS2.8-BR, symbol MerlynActionCam:RT9193-18GB
- added U7: ICS43434, easyeda2kicad:MIC-SMD_6P-L3.5-W2.7-P0.90-BL, symbol MerlynActionCam:ICS-43434_C5656610
- added U8: BMI270, easyeda2kicad:LGA-14_L3.0-W2.5-P0.50-BR, symbol MerlynActionCam:BMI270
- added U9: INMP441, easyeda2kicad:MIC-SMD_INMP441, symbol MerlynActionCam:INMP441
- added X1: 24MHz, easyeda2kicad:CRYSTAL-SMD_4P-L2.0-W1.6-BL, symbol MerlynActionCam:T201624MBBCE2X
- BT1: footprint (none) -> easyeda2kicad:Battery
- BT2: now not fitted
- JP1: footprint (none) -> easyeda2kicad:SolderJumper-2_P1.3mm_Open_TrianglePad1.0x1.5mm
- TP1, TP2: footprint (none) -> easyeda2kicad:TestPoint
- renumbered 1 to U12
Connections:
- net +1V0: now also U12.115 (VDD), U12.120 (VDD), U12.23 (VDD), U12.44 (DVDD_DDR), U12.45 (VDD), U12.47 (VDD), U12.87 (VDD), U12.88 (VDD), U12.96 (VDD)
- net +1V5: now also U12.40 (AVDDIO_DRAM), U12.41 (AVDDIO_DATA), U12.46 (VDDIO_DATA), U12.48 (VDDIO_MCLK), U12.49 (VDDIO_DRAM)
- net +3V3: now also R25.2, U12.116 (AVDD_XTAL), U12.127 (VDDP_0), U12.24 (VDD_ETH), U12.29 (AVDD3P3_USB), U12.32 (AVDD_AUD), U12.42 (AVDD_PLL), U12.65 (AVDD_NODIE), U12.72 (AVDD_PM_SPI), U12.84 (AVDD_RTC), U12.89 (VDDP_1), C20.1, C21.1, C22.1, C23.1, C24.1, C26.1, C28.1, C31.1, C32.1, C35.1, C36.1, R31.2, R35.1, U10.8 (VCC), U11.4 (VDD), U6.1 (VIN), U6.3 (EN), U7.5 (VDD), U8.12 (CSB), U8.5 (VDDIO), U8.8 (VDD), U9.7 (VDD), U9.8 (CHIPEN)
- net GND: now also CN1.31, CN1.32, CN1.33, CN1.34, U12.129 (EP), U12.34 (AUD_VRM_ADC), C18.2, C19.2, C20.2, C21.2, C22.2, C23.2, C24.2, C25.2, C26.2, C27.2, C28.2, C29.2, C30.1, C31.2, C32.2, C33.2, C34.1, C36.2, H1.2 (GND), R26.1, R27.2, R28.1, R29.2, R30.2, R34.1, R36.2, R37.2, U10.4 (GND), U11.10 (GND), U11.11 (GND), U11.12 (GND), U11.13 (GND), U11.6 (VSS), U6.2 (GND), U7.2 (LR), U7.3 (GND), U8.1 (SDO), U8.6 (GNDIO), U8.7 (GND), U9.4 (L/R), U9.5 (GND), U9.6 (GND), U9.9 (GND), X1.2 (GND), X1.4 (GND)
- net MIPI_D0+: now also U12.108 (SR0_IO10); no longer U12.100 (SR0_IO2)
- net MIPI_D0-: now also U12.109 (SR0_IO11); no longer U12.101 (SR0_IO3)
- net MIPI_D1+: now also U12.106 (SR0_IO8); no longer U12.102 (SR0_IO4)
- net MIPI_D1-: now also U12.107 (SR0_IO9); no longer U12.103 (SR0_IO5)
- net MIPI_D2+: now also U12.102 (SR0_IO4); no longer U12.106 (SR0_IO8)
- net MIPI_D2-: now also U12.103 (SR0_IO5); no longer U12.107 (SR0_IO9)
- net MIPI_D3+: now also U12.100 (SR0_IO2); no longer U12.108 (SR0_IO10)
- net MIPI_D3-: now also U12.101 (SR0_IO3); no longer U12.109 (SR0_IO11)
- net REC_SIGNAL: now also U12.57 (PM_GPIO1)
- net SCL: now also R32.1
- net SDA: now also R33.1
- net +5-14VRP: now reaches BT2.1 (+), Q2.3 (D)
- net +5-14VRP: now also H1.1 (5v)
- net at LED1.1 (K): now also U12.56 (PM_GPIO0)
- net SPI_SCK: now reaches U12.1 (SPI_CK)
- net SPI_SCK: now also U10.6 (CLK)
- net SD_CLK: now reaches U12.10 (SD0_CLK)
- net SD_CLK: now also U11.5 (CLK)
- net SD_CMD: now reaches U12.11 (SD0_CMD)
- net SD_CMD: now also U11.3 (CMD)
- net at U12.117 (XTAL_IN): now also C27.1, X1.1
- net at U12.118 (XTAL_OUT): now also C25.1, X1.3
- net SD_DATA3: now reaches U12.12 (SD0_D3)
- net SD_DATA3: now also U11.2 (CD/DATA3)
- net SPI_CZ: now reaches U12.128 (SPI_CZ)
- net SPI_CZ: now also U10.1 (~{CS})
- net SD_DATA2: now reaches U12.13 (SD0_D2)
- net SD_DATA2: now also U11.1 (DATA2)
- net I2S0_BCK: now reaches U12.15 (I2S0_BCK)
- net I2S0_BCK: now also U7.4 (SCK), U9.1 (SCK)
- net I2S0_WCK: now reaches U12.16 (I2S0_WCK)
- net I2S0_WCK: now also U7.1 (WS), U9.3 (WS)
- net I2S0_DI: now reaches U12.17 (I2S0_DI)
- net I2S0_DI: now also R26.2, R27.1, U7.6 (SD), U9.2 (SD)
- net SPI_SDI: now reaches U12.2 (SPI_DI)
- net SPI_SDI: now also U10.5 (DI)
- net SPI_SDO: now reaches U12.3 (SPI_DO)
- net SPI_SDO: now also U10.2 (DO)
- net at U12.33 (AUD_AVG): now also C29.1
- net SPI_WPZ: now reaches U12.4 (SPI_WPZ)
- net SPI_WPZ: now also U10.3 (IO2)
- net at U12.43 (DVDD_DDR_RX): now also C34.2
- net SPI_HLD: now reaches U12.5 (SPI_HLD)
- net SPI_HLD: now also U10.7 (IO3)
- net at U12.50 (PM_UART_RX): now also TP4.1
- net at U12.51 (PM_UART_TX): now also TP3.1
- net PM_I2CM_SCL: now reaches U12.54 (PM_I2CM_SCL)
- net PM_I2CM_SCL: now also U8.13 (SCX)
- net PM_I2CM_SDA: now reaches U12.55 (PM_I2CM_SDA)
- net PM_I2CM_SDA: now also U8.14 (SDX)
- net at U12.62 (PM_GPIO6): now also R30.1
- net at U12.64 (PM_GPIO8): now also R31.1
- net at U12.67 (PM_SPI_CK): now also R35.2
- net SD_CDZ: now reaches U12.7 (SD0_CDZ)
- net SD_CDZ: now also R28.2, U11.9 (CD)
- net at U12.70 (PM_SPI_WPZ): now also R34.2
- net at U12.73 (DVDD_NODIE): now also C30.2
- net SD_DATA1: now reaches U12.8 (SD0_D1)
- net SD_DATA1: now also U11.8 (DAT1)
- net at U12.83 (RESET): now also C35.2, R29.1
- net at U12.85 (XTAL_IN_32K): now also R37.1
- net at U12.86 (XTAL_OUT_32K): now also R36.1
- net SD_DATA0: now reaches U12.9 (SD0_D0)
- net SD_DATA0: now also U11.7 (DAT0)
- net at U12.90 (FUART_RX): now also H1.3 (RX)
- net at U12.91 (FUART_TX): now also H1.4 (TX)
- net +1V8: now reaches U12.97 (VDDP_2A)
- net +1V8: now also C19.1, C33.1, R32.2, R33.2, R38.2, U6.5 (VOUT)
- net at CN1.9: now also R38.1
- new net: C18.1, U6.4 (BP)
- no-connect marks 21 -> 77
Other:
- note added: "1.8V Regulator"
- note added: "30P Mezzanine Camera Connector"
- note added: "IMU"
- note added: "Microphone"
- note added: "NOR Flash"
- note added: "SD Card Connector"
- moved on the sheet: CN1, LED1, R25

Commit message: checkpoint
Parts:
- added C37, C38, C39, C40, C41, C42, C43, C46, C47, C48, C49, C51, C52, C53, C54, C55, C56, C57: 0.1uF, Capacitor_SMD:C_0402_1005Metric, symbol Device:C_Small
- added C44, C45, C50, C58, C59, C60, C61: 10uF, Capacitor_SMD:C_0603_1608Metric, symbol Device:C_Small
Connections:
- net +1V0: now also C50.1, C51.1, C52.1, C53.1, C54.1, C55.1, C56.1, C57.1, C59.1, C60.1, C61.1
- net +1V5: now also C45.1, C46.1, C47.1, C48.1, C49.1
- net +3V3: now also C37.1, C38.1, C39.1, C40.1, C41.1, C42.1, C43.1, C44.1, C58.1
- net GND: now also C37.2, C38.2, C39.2, C40.2, C41.2, C42.2, C43.2, C44.2, C45.2, C46.2, C47.2, C48.2, C49.2, C50.2, C51.2, C52.2, C53.2, C54.2, C55.2, C56.2, C57.2, C58.2, C59.2, C60.2, C61.2

Commit message: checkpoint
Parts:
- removed C22: 0.1uF, Capacitor_SMD:C_0402_1005Metric, symbol Device:C_Small
- removed R27: 100k, Resistor_SMD:R_0402_1005Metric, symbol Device:R_Small
Connections:
- net at C27.1, U12.117 (XTAL_IN): now also X1.3; no longer X1.1
- net at C25.1, U12.118 (XTAL_OUT): now also X1.1; no longer X1.3
Other:
- moved on the sheet: X1
Changed lines of the file:
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@@
 	)
 	(junction
-		(at 269.24 92.71)
-		(diameter 0)
-		(color 0 0 0 0)
-	)
-	(junction
 		(at 516.89 49.53)
 		(diameter 0)
@@
 	)
 	(junction
-		(at 269.24 97.79)
-		(diameter 0)
-		(color 0 0 0 0)
-	)
-	(junction
 		(at 207.01 166.37)
 		(diameter 0)
@@
 	)
 	(junction
-		(at 242.57 99.06)
-		(diameter 0)
-		(color 0 0 0 0)
-	)
-	(junction
 		(at 440.69 120.65)
 		(diameter 0)
@@
 	(wire
 		(pts
-			(xy 240.03 88.9) (xy 240.03 93.98)
-		)
-		(stroke
-			(width 0)
-			(type default)
-		)
-	)
-	(wire
-		(pts
 			(xy 241.3 381) (xy 240.03 381)
 		)
@@
 	(wire
 		(pts
-			(xy 269.24 97.79) (xy 269.24 99.06)
-		)
-		(stroke
-			(width 0)
-			(type default)
-		)
-	)
-	(wire
-		(pts
 			(xy 226.06 171.45) (xy 232.41 171.45)
 		)
@@
 	(wire
 		(pts
-			(xy 240.03 99.06) (xy 242.57 99.06)
-		)
-		(stroke
-			(width 0)
-			(type default)
-		)
-	)
-	(wire
-		(pts
 			(xy 382.27 102.87) (xy 384.81 102.87)
 		)
@@
 	(wire
 		(pts
-			(xy 269.24 97.79) (xy 265.43 97.79)
-		)
-		(stroke
-			(width 0)
-			(type default)
-		)
-	)
-	(wire
-		(pts
 			(xy 212.09 193.04) (xy 214.63 193.04)
 		)
@@
 	)
 	(symbol
-		(lib_id "Device:R_Small")
-		(at 240.03 96.52 0)
-		(mirror y)
-		(unit 1)
-		(exclude_from_sim no)
-		(in_bom yes)
-		(on_board yes)
-		(dnp no)
-		(property "Reference" "R27"
-			(at 239.014 95.504 0)
-			(effects
-				(font
-					(size 1.27 1.27)
-				)
-				(justify left)
-			)
-		)
-		(property "Value" "100k"
-			(at 239.014 97.282 0)
-			(effects
-				(font
-					(size 1.27 1.27)
-				)
-				(justify left)
-			)
-		)
-		(property "Footprint" "Resistor_SMD:R_0402_1005Metric"
-			(at 240.03 96.52 0)
-			(effects
-				(font
-					(size 1.27 1.27)
-				)
-				(hide yes)
-			)
-		)
-		(property "Datasheet" "100k, 0402"
-			(at 240.03 96.52 0)
-			(effects
-				(font
-					(size 1.27 1.27)
-				)
-				(hide yes)
-			)
-		)
-		(property "Description" "Resistor, small symbol"
-			(at 240.03 96.52 0)
-			(effects
-				(font
-					(size 1.27 1.27)
-				)
-				(hide yes)
-			)
-		)
-		(property "LCSC Part" "C25741"
-			(at 240.03 96.52 0)
-			(effects
-				(font
-					(size 1.27 1.27)
-				)
-				(hide yes)
-			)
-		)
-		(pin "2"
-		)
-		(pin "1"
-		)
-		(instances
-			(project "MerlynActionCam"
-				(path "/87d09840-694d-4014-a159-e691c619b33e"
-					(reference "R27")
-					(unit 1)
-				)
-			)
-		)
-	)
-	(symbol
 		(lib_id "power:GND")
 		(at 439.42 95.25 90)
@@
 	(symbol
 		(lib_id "MerlynActionCam:T201624MBBCE2X")
-		(at 261.62 370.84 270)
+		(at 261.62 370.84 90)
 		(unit 1)
 		(exclude_from_sim no)
@@
 		(dnp no)
 		(property "Reference" "X1"
-			(at 268.224 373.634 90)
+			(at 268.478 372.872 90)
 			(effects
 				(font
@@
 		)
 		(property "Value" "24MHz"
-			(at 270.002 375.158 90)
+			(at 270.256 374.65 90)
 			(effects
 				(font
@@
 		)
 		(property "Footprint" "easyeda2kicad:CRYSTAL-SMD_4P-L2.0-W1.6-BL"
-			(at 251.46 370.84 0)
+			(at 271.78 370.84 0)
 			(effects
 				(font
@@
 		)
 		(property "Datasheet" "https://www.lcsc.com/datasheet/C7303340.pdf"
-			(at 248.92 370.84 0)
+			(at 274.32 370.84 0)
 			(effects
 				(font
@@
 		)
 		(property "Manufacturer" "YJX(雅晶鑫)"
-			(at 246.38 370.84 0)
+			(at 276.86 370.84 0)
 			(effects
 				(font
@@
 		)
 		(property "MPN" "T201624MBBCE2X"
-			(at 243.84 370.84 0)
+			(at 279.4 370.84 0)
 			(effects
 				(font
@@
 		)
 		(property "LCSC Part" "C7303340"
-			(at 241.3 370.84 0)
+			(at 281.94 370.84 0)
 			(effects
 				(font
@@
 	(symbol
 		(lib_id "power:GND")
-		(at 269.24 99.06 0)
+		(at 265.43 97.79 0)
 		(unit 1)
 		(exclude_from_sim no)
@@
 		(dnp no)
 		(property "Reference" "#PWR067"
-			(at 269.24 105.41 0)
+			(at 265.43 104.14 0)
 			(effects
 				(font
@@
 		)
 		(property "Value" "GND"
-			(at 269.24 102.616 0)
+			(at 265.43 101.346 0)
 			(effects
 				(font
@@
 		)
 		(property "Footprint" ""
-			(at 269.24 99.06 0)
+			(at 265.43 97.79 0)
 			(effects
 				(font
@@
 		)
 		(property "Datasheet" ""
-			(at 269.24 99.06 0)
+			(at 265.43 97.79 0)
 			(effects
 				(font
@@
 		)
 		(property "Description" "Power symbol creates a global label with name \"GND\" , ground"
-			(at 269.24 99.06 0)
+			(at 265.43 97.79 0)
 			(effects
 				(font
@@
 					(unit 1)
 				)
-			)
-		)
-	)
-	(symbol
-		(lib_id "Device:C_Small")
-		(at 269.24 95.25 0)
-		(unit 1)
-		(exclude_from_sim no)
-		(in_bom yes)
-		(on_board yes)
-		(dnp no)
-		(property "Reference" "C22"
-			(at 271.018 94.488 0)
-			(effects
-				(font
-					(size 1.27 1.27)
-				)
-				(justify left)
-			)
-		)
-		(property "Value" "0.1uF"
-			(at 271.018 96.266 0)
-			(effects
-				(font
-					(size 1.27 1.27)
-				)
-				(justify left)
-			)
-		)
-		(property "Footprint" "Capacitor_SMD:C_0402_1005Metric"
-			(at 269.24 95.25 0)
-			(effects
-				(font
-					(size 1.27 1.27)
-				)
-				(hide yes)
-			)
-		)
-		(property "Datasheet" "0.1uF, 0402, 50V"
-			(at 269.24 95.25 0)
-			(effects
-				(font
-					(size 1.27 1.27)
-				)
-				(hide yes)
-			)
-		)
-		(property "Description" "Unpolarized capacitor, small symbol"
-			(at 269.24 95.25 0)
-			(effects
-				(font
-					(size 1.27 1.27)
-				)
-				(hide yes)
-			)
-		)
-		(property "LCSC Part" "C307331"
-			(at 269.24 95.25 0)
-			(effects
-				(font
-					(size 1.27 1.27)
-				)
-				(hide yes)
-			)
-		)
-		(pin "1"
-		)
-		(pin "2"
-		)
-		(instances
-			(project "MerlynActionCam"
-				(path "/87d09840-694d-4014-a159-e691c619b33e"
-					(reference "C22")
-					(unit 1)
-				)

Commit message: checkpoint
Parts:
- removed C59: 10uF, Capacitor_SMD:C_0603_1608Metric, symbol Device:C_Small
- added C22: 10uF, Capacitor_SMD:C_0603_1608Metric, symbol Device:C_Small
- added R27: 100R, Resistor_SMD:R_0402_1005Metric, symbol Device:R_Small
Connections:
- net +3V3: now also C22.1
- net GND: now also C22.2, R27.1; no longer C29.2, U12.34 (AUD_VRM_ADC)
- new net: C29.2, R27.2, U12.34 (AUD_VRM_ADC)
Other:
- moved on the sheet: C60, C61
