File: PCB/MerlynCAM.kicad_pcb (KiCad board)
At the start: 4 copper layers, 45 x 38 mm, 135 parts, among them CN1 OK-10F030-04, Q1 AO3401A, Q2 AO3401A, Q3 AO3401A, SW1 TS24CA, U1 TPS63802DLAR, U10 W25Q128JVSIQTR, U11 TF-115-BCP9, U2 BQ25606RGER, U3 RT8097CHGE, U4 RT8097CHGE, U5 CH32V003F4U6, U6 RT9193-18GB, U7 ICS43434, U8 BMI270, U9 INMP441, X1 24MHz

Commit message: Updated PCB to Rev 2
Parts:
- added JP2: Bypass, easyeda2kicad:SolderJumper-2_P1.3mm_Open_TrianglePad1.0x1.5mm, B.Cu at (198.5, 87.0)
- added R39: 5.1k, Resistor_SMD:R_0402_1005Metric, B.Cu at (218.3, 110.0)
- added R40: 5.1k, Resistor_SMD:R_0402_1005Metric, B.Cu at (217.3, 110.0)
- added TP10: 3V3, easyeda2kicad:TestPoint, B.Cu at (220.9, 84.6)
- added TP11: 1V8, easyeda2kicad:TestPoint, B.Cu at (205.8, 89.8)
- added TP12: GND, easyeda2kicad:TestPoint, B.Cu at (187.7, 104.1)
- added TP13: ETH_RN, easyeda2kicad:TestPoint, F.Cu at (207.6, 103.2)
- added TP14: ETH_RP, easyeda2kicad:TestPoint, F.Cu at (205.5, 104.0)
- added TP15: ETH_TN, easyeda2kicad:TestPoint, B.Cu at (204.1, 105.8)
- added TP16: ETH_TP, easyeda2kicad:TestPoint, B.Cu at (205.9, 105.8)
- added TP5: USBD+, easyeda2kicad:TestPoint, B.Cu at (192.3, 104.1)
- added TP6: USBD-, easyeda2kicad:TestPoint, B.Cu at (194.6, 104.1)
- added TP7: +5-14V, easyeda2kicad:TestPoint, B.Cu at (190.0, 104.1)
- added TP8: 1V0, easyeda2kicad:TestPoint, B.Cu at (201.1, 86.5)
- added TP9: 1V5, easyeda2kicad:TestPoint, B.Cu at (212.2, 85.2)
- C42, C44, R32, R33, R38: moved to B.Cu
- moved C44 10.0 mm to (223.6, 91.8), turned to 90 degrees
- moved C42 9.95 mm to (223.7, 93.8), turned to 0 degrees
- moved R32 8.02 mm to (212.9, 89.3), turned to 90 degrees
- moved R38 6.85 mm to (221.5, 93.9), turned to 0 degrees
- moved R33 5.09 mm to (213.9, 89.3), turned to 90 degrees
- moved C61 2.63 mm to (214.9, 96.4), turned to 0 degrees
- moved CN1 0.30 mm to (218.5, 91.1), turned to 0 degrees
Connections:
- CN1 pad 16: MIPI_D0- -> MIPI_D0+
- CN1 pad 17: MIPI_D0+ -> MIPI_D0-
- U12 pad 100: MIPI_D3+ -> MIPI_D0+
- U12 pad 101: MIPI_D3- -> MIPI_D0-
- U12 pad 102: MIPI_D2+ -> MIPI_D1+
- U12 pad 103: MIPI_D2- -> MIPI_D1-
- U12 pad 106: MIPI_D1+ -> MIPI_D2+
- U12 pad 107: MIPI_D1- -> MIPI_D2-
- U12 pad 108: MIPI_D0+ -> MIPI_D3+
- U12 pad 109: MIPI_D0- -> MIPI_D3-
- U12 pad 25: unconnected-(U12-ETH_RN-Pad25) -> Net-(U12-ETH_RN)
- U12 pad 26: unconnected-(U12-ETH_RP-Pad26) -> Net-(U12-ETH_RP)
- U12 pad 27: unconnected-(U12-ETH_TN-Pad27) -> Net-(U12-ETH_TN)
- U12 pad 28: unconnected-(U12-ETH_TP-Pad28) -> Net-(U12-ETH_TP)
Routing:
- net Net-(JP2-B): track 38.0 -> 51.1 mm, vias 2 -> 3
- net +1V8: track 42.9 -> 34.4 mm
- net +3V3: track 174.9 -> 181.0 mm, vias 19 -> 20
- net Net-(U12-ETH_TN): track 0.00 -> 5.80 mm, vias 0 -> 1
- net GND: track 81.3 -> 76.5 mm, vias 115 -> 132
- net MIPI_MCLK: track 9.01 -> 13.2 mm
- net Net-(U12-ETH_TP): track 0.00 -> 3.95 mm, vias 0 -> 1
- net Net-(U12-ETH_RP): track 0.00 -> 3.81 mm
- net MIPI_CLK-: track 2.23 -> 5.34 mm, vias 0 -> 2
- net MIPI_D1-: track 2.18 -> 5.25 mm, vias 0 -> 2
- net MIPI_D1+: track 2.16 -> 5.16 mm, vias 0 -> 2
- net MIPI_CLK+: track 2.25 -> 5.25 mm, vias 0 -> 2
- net MIPI_D0+: track 2.37 -> 5.27 mm, vias 0 -> 2
- net MIPI_D0-: track 2.39 -> 5.27 mm, vias 0 -> 2
- net SDA: track 11.8 -> 9.04 mm, vias 2 -> 1
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Other:
- board text added: "1V0"
- board text added: "1V5"
- board text added: "1V8"
- board text added: "3V3"
- board text added: "5-14V"
- board text added: "BYPS"
- board text added: "DISAB"
- board text added: "ERN"
- board text added: "ERP"
- board text added: "ETN"
- board text added: "ETP"
- board text added: "GND"
- board text added: "MerlynCam"
- board text added: "PWR"
- board text added: "Rev 2"
- board text added: "USB_DN"
- board text added: "USB_DP"
