File: PCB/MerlynCAM.kicad_sch (KiCad schematic)
At the start: 132 parts, among them CN1 OK-10F030-04, Q1 AO3401A, Q2 AO3401A, Q3 AO3401A, SW1 TS24CA, U1 TPS63802DLAR, U10 W25Q128JVSIQTR, U11 TF-115-BCP9, U2 BQ25606RGER, U3 RT8097CHGE, U4 RT8097CHGE, U5 CH32V003F4U6, U6 RT9193-18GB, U7 ICS43434, U8 BMI270, U9 INMP441, X1 24MHz

Commit message: Updated PCB to Rev 2
Parts:
- added JP2: Bypass, easyeda2kicad:SolderJumper-2_P1.3mm_Open_TrianglePad1.0x1.5mm, symbol Jumper:SolderJumper_2_Open
- added R39, R40: 5.1k, Resistor_SMD:R_0402_1005Metric, symbol Device:R_Small
- added TP10: 3V3, easyeda2kicad:TestPoint, symbol Connector:TestPoint
- added TP11: 1V8, easyeda2kicad:TestPoint, symbol Connector:TestPoint
- added TP12: GND, easyeda2kicad:TestPoint, symbol Connector:TestPoint
- added TP13: ETH_RN, easyeda2kicad:TestPoint, symbol Connector:TestPoint
- added TP14: ETH_RP, easyeda2kicad:TestPoint, symbol Connector:TestPoint
- added TP15: ETH_TN, easyeda2kicad:TestPoint, symbol Connector:TestPoint
- added TP16: ETH_TP, easyeda2kicad:TestPoint, symbol Connector:TestPoint
- added TP5: USBD+, easyeda2kicad:TestPoint, symbol Connector:TestPoint
- added TP6: USBD-, easyeda2kicad:TestPoint, symbol Connector:TestPoint
- added TP7: +5-14V, easyeda2kicad:TestPoint, symbol Connector:TestPoint
- added TP8: 1V0, easyeda2kicad:TestPoint, symbol Connector:TestPoint
- added TP9: 1V5, easyeda2kicad:TestPoint, symbol Connector:TestPoint
Connections:
- net +1V0: now also TP8.1
- net +1V5: now also TP9.1
- net +1V8: now also TP11.1
- net +3V3: now also R39.2, R40.2, TP10.1
- net +5-14V: now also TP7.1
- net D+: now also TP5.1
- net D-: now also TP6.1
- net GND: now also JP2.1 (A), TP12.1
- net MIPI_D0+: now also CN1.16, U12.100 (SR0_IO2); no longer CN1.17, U12.108 (SR0_IO10)
- net MIPI_D0-: now also CN1.17, U12.101 (SR0_IO3); no longer CN1.16, U12.109 (SR0_IO11)
- net MIPI_D1+: now also U12.102 (SR0_IO4); no longer U12.106 (SR0_IO8)
- net MIPI_D1-: now also U12.103 (SR0_IO5); no longer U12.107 (SR0_IO9)
- net MIPI_D2+: now also U12.106 (SR0_IO8); no longer U12.102 (SR0_IO4)
- net MIPI_D2-: now also U12.107 (SR0_IO9); no longer U12.103 (SR0_IO5)
- net MIPI_D3+: now also U12.108 (SR0_IO10); no longer U12.100 (SR0_IO2)
- net MIPI_D3-: now also U12.109 (SR0_IO11); no longer U12.101 (SR0_IO3)
- net PM_I2CM_SCL: now also R39.1
- net PM_I2CM_SDA: now also R40.1
- net at Q3.1 (G), R18.2, R19.1: now also JP2.2 (B)
- net at U12.25 (ETH_RN): now also TP13.1
- net at U12.26 (ETH_RP): now also TP14.1
- net at U12.27 (ETH_TN): now also TP15.1
- net at U12.28 (ETH_TP): now also TP16.1
- no-connect marks 77 -> 73
Other:
- moved on the sheet: BT1, BT2, C1, C10, C11, C12, C13, C14, C15, C16, C17, C18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
